Commit message: XACRO refactorization: Making robots and objects strict and applicable format
Signed-off-by: silanus23 <berkantali23@outlook.com>

File: hold_and_weld_description/urdf/end_effectors/gripper_prefix.xacro (robot description, xacro)
@@ -72,4 +72,5 @@
       <axis xyz="0 1 0"/>
       <limit lower="0.0" upper="0.15" effort="100" velocity="0.1"/>
+      <dynamics damping="1.0" friction="2.0"/>
     </joint>
     <joint name="${prefix}right_finger_joint" type="prismatic">
@@ -79,4 +80,5 @@
       <axis xyz="0 -1 0"/>
       <limit lower="0.0" upper="0.15" effort="100" velocity="0.1"/>
+      <dynamics damping="1.0" friction="2.0"/>
     </joint>
     <gazebo reference="${prefix}gripper_base">

File: hold_and_weld_description/urdf/environment/cube.urdf.xacro (robot description, xacro)
@@ -1,6 +1,6 @@
 <?xml version="1.0"?>
-<robot xmlns:xacro="http://ros.org/wiki/xacro" name="cube">
+<robot xmlns:xacro="http://ros.org/wiki/xacro" name="child_link">
   <xacro:property name="cube_size" value="0.25"/>
-  <link name="target_cube">
+  <link name="child_link">
     <visual>
       <geometry>
@@ -23,5 +23,5 @@
   </link>
   <!-- Gazebo properties for the cube -->
-  <gazebo reference="target_cube">
+  <gazebo reference="child_link">
     <visual>
       <material>

File: hold_and_weld_description/urdf/environment/workpiece.urdf.xacro (robot description, xacro)
@@ -1,9 +1,9 @@
 <?xml version="1.0"?>
-<robot xmlns:xacro="http://ros.org/wiki/xacro" name="workpiece">
+<robot xmlns:xacro="http://ros.org/wiki/xacro" name="base_link">
   <!-- Workpiece dimensions -->
   <xacro:property name="length" value="0.80"/>  <!-- 80cm -->
   <xacro:property name="width" value="0.40"/>   <!-- 40cm -->
   <xacro:property name="height" value="0.30"/>  <!-- 30cm -->
-  <link name="workpiece_body">
+  <link name="base_link">
     <visual>
       <geometry>
@@ -26,5 +26,5 @@
   </link>
   <!-- Gazebo properties for the workpiece -->
-  <gazebo reference="workpiece_body">
+  <gazebo reference="base_link">
     <visual>
       <material>
