Commit message: Debugging and styling sampler package
Signed-off-by: silanus23 <berkantali23@outlook.com>

File: hold_and_weld_gripper_sampler/config/test_gripper.urdf (robot description, URDF)
Before this commit: robot test_gripper, 3 links, 2 joints
Joints:
- joint left_finger_joint: origin xyz=0 0.03 -0.02 rpy=0 0 0 -> xyz=0 0.03 0.02 rpy=0 0 0
- joint right_finger_joint: origin xyz=0 -0.03 -0.02 rpy=0 0 0 -> xyz=0 -0.03 0.02 rpy=0 0 0
