Commit message: Refine planning package
Signed-off-by: silanus23 <berkantali23@outlook.com>

File: hold_and_weld_description/urdf/environment/cube.urdf.xacro (robot description, xacro)
@@ -7,6 +7,6 @@
         <box size="${cube_size} ${cube_size} ${cube_size}"/>
       </geometry>
-      <material name="red">
-        <color rgba="1 0 0 1"/>
+      <material name="blue">
+        <color rgba="0 0.45 0.9 1"/>
       </material>
     </visual>
@@ -26,6 +26,6 @@
     <visual>
       <material>
-        <ambient>1 0 0 1</ambient>
-        <diffuse>1 0 0 1</diffuse>
+        <ambient>0 0.45 0.9 1</ambient>
+        <diffuse>0 0.45 0.9 1</diffuse>
         <specular>0.5 0.5 0.5 1</specular>
       </material>
