Commit message: Now system bringup launch handles spawning welder in safe position and dual robot coordinator became moveit agnostic. A long time TODO has been handled.
Signed-off-by: silanus23 <berkantali23@outlook.com>

File: hold_and_weld_description/urdf/dual_robot.xacro (robot description, xacro)
@@ -3,4 +3,12 @@
   <xacro:arg name="controller_config_file" default=""/>
   <xacro:property name="controller_config_file" value="$(arg controller_config_file)"/>
+  <!-- Robot2 initial joint positions (radians). Populated by sim_gazebo.launch.py
+       from welding.yaml safety_pose so the welder spawns collision-free. -->
+  <xacro:arg name="robot2_initial_pos_j1" default="0"/>
+  <xacro:arg name="robot2_initial_pos_j2" default="0"/>
+  <xacro:arg name="robot2_initial_pos_j3" default="0"/>
+  <xacro:arg name="robot2_initial_pos_j4" default="0"/>
+  <xacro:arg name="robot2_initial_pos_j5" default="0"/>
+  <xacro:arg name="robot2_initial_pos_j6" default="0"/>
   <!-- Include all macro files -->
   <xacro:include filename="$(find hold_and_weld_description)/urdf/extra_axis/linear_rail_prefix.xacro"/>
@@ -19,5 +27,11 @@
   </joint>
   <!-- Robot 2: Welder System (standalone) -->
-  <xacro:gp25_arm_macro parent="world" prefix="robot2_" x="2.2" y="-0.5" z="0" yaw='3.14159'/>
+  <xacro:gp25_arm_macro parent="world" prefix="robot2_" x="2.2" y="-0.5" z="0" yaw='3.14159'
+    initial_pos_j1="$(arg robot2_initial_pos_j1)"
+    initial_pos_j2="$(arg robot2_initial_pos_j2)"
+    initial_pos_j3="$(arg robot2_initial_pos_j3)"
+    initial_pos_j4="$(arg robot2_initial_pos_j4)"
+    initial_pos_j5="$(arg robot2_initial_pos_j5)"
+    initial_pos_j6="$(arg robot2_initial_pos_j6)"/>
   <xacro:welding_torch_macro prefix="robot2_"/>
   <joint name="robot2_tool0_to_torch" type="fixed">

File: hold_and_weld_description/urdf/robots/gp25_arm_prefix.xacro (robot description, xacro)
@@ -1,5 +1,7 @@
 <?xml version="1.0"?>
 <robot xmlns:xacro="http://ros.org/wiki/xacro" name="gp25_arm_macro">
-  <xacro:macro name="gp25_arm_macro" params="parent prefix x:=0 y:=0 z:=0 roll:=0 pitch:=0 yaw:=0">
+  <xacro:macro name="gp25_arm_macro" params="parent prefix x:=0 y:=0 z:=0 roll:=0 pitch:=0 yaw:=0
+               initial_pos_j1:=0 initial_pos_j2:=0 initial_pos_j3:=0
+               initial_pos_j4:=0 initial_pos_j5:=0 initial_pos_j6:=0">
     <joint name="${prefix}base_joint" type="fixed">
       <parent link="${parent}"/>
@@ -251,5 +253,7 @@
           <param name="max">3.14159</param>
         </command_interface>
-        <state_interface name="position"/>
+        <state_interface name="position">
+          <param name="initial_value">${initial_pos_j1}</param>
+        </state_interface>
         <state_interface name="velocity"/>
       </joint>
@@ -259,5 +263,7 @@
           <param name="max">2.70526</param>
         </command_interface>
-        <state_interface name="position"/>
+        <state_interface name="position">
+          <param name="initial_value">${initial_pos_j2}</param>
+        </state_interface>
         <state_interface name="velocity"/>
       </joint>
@@ -267,5 +273,7 @@
           <param name="max">2.79253</param>
         </command_interface>
-        <state_interface name="position"/>
+        <state_interface name="position">
+          <param name="initial_value">${initial_pos_j3}</param>
+        </state_interface>
         <state_interface name="velocity"/>
       </joint>
@@ -275,5 +283,7 @@
           <param name="max">3.49066</param>
         </command_interface>
-        <state_interface name="position"/>
+        <state_interface name="position">
+          <param name="initial_value">${initial_pos_j4}</param>
+        </state_interface>
         <state_interface name="velocity"/>
       </joint>
@@ -283,5 +293,7 @@
           <param name="max">2.61799</param>
         </command_interface>
-        <state_interface name="position"/>
+        <state_interface name="position">
+          <param name="initial_value">${initial_pos_j5}</param>
+        </state_interface>
         <state_interface name="velocity"/>
       </joint>
@@ -291,5 +303,7 @@
           <param name="max">7.94163</param>
         </command_interface>
-        <state_interface name="position"/>
+        <state_interface name="position">
+          <param name="initial_value">${initial_pos_j6}</param>
+        </state_interface>
         <state_interface name="velocity"/>
       </joint>

Commit message: updating robot to ar2010
Signed-off-by: silanus23 <berkantali23@outlook.com>

File: hold_and_weld_description/urdf/dual_robot.xacro (robot description, xacro)
@@ -1,4 +1,4 @@
 <?xml version="1.0"?>
-<robot xmlns:xacro="http://ros.org/wiki/xacro" name="dual_gp25_system">
+<robot xmlns:xacro="http://ros.org/wiki/xacro" name="dual_robot_system">
   <xacro:arg name="controller_config_file" default=""/>
   <xacro:property name="controller_config_file" value="$(arg controller_config_file)"/>
@@ -13,5 +13,6 @@
   <!-- Include all macro files -->
   <xacro:include filename="$(find hold_and_weld_description)/urdf/extra_axis/linear_rail_prefix.xacro"/>
-  <xacro:include filename="$(find hold_and_weld_description)/urdf/robots/gp25_arm_prefix.xacro"/>
+  <xacro:include filename="$(find hold_and_weld_description)/urdf/robots/gp25_arm_prefix.xacro"/> <!-- Robot1 (gripper) -->
+  <xacro:include filename="$(find hold_and_weld_description)/urdf/robots/ar2010_arm_prefix.xacro"/> <!-- Robot2 (welder) -->
   <xacro:include filename="$(find hold_and_weld_description)/urdf/end_effectors/gripper_prefix.xacro"/>
   <xacro:include filename="$(find hold_and_weld_description)/urdf/end_effectors/welding_torch_prefix.xacro"/>
@@ -19,5 +20,5 @@
   <!-- Robot 1: Gripper System with Rail -->
   <xacro:linear_rail_macro parent="world" prefix="robot1_"/>
-  <xacro:gp25_arm_macro parent="robot1_rail_carriage" prefix="robot1_"/>
+  <xacro:gp25_arm_macro parent="robot1_rail_carriage" prefix="robot1_" controller_config_file="${controller_config_file}"/>
   <xacro:gripper_macro prefix="robot1_"/>
   <joint name="robot1_tool0_to_gripper" type="fixed">
@@ -27,5 +28,5 @@
   </joint>
   <!-- Robot 2: Welder System (standalone) -->
-  <xacro:gp25_arm_macro parent="world" prefix="robot2_" x="2.2" y="-0.5" z="0" yaw='3.14159'
+  <xacro:ar2010_arm_macro parent="world" prefix="robot2_" x="2.2" y="-0.5" z="0" yaw='3.14159'
     initial_pos_j1="$(arg robot2_initial_pos_j1)"
     initial_pos_j2="$(arg robot2_initial_pos_j2)"
@@ -33,5 +34,6 @@
     initial_pos_j4="$(arg robot2_initial_pos_j4)"
     initial_pos_j5="$(arg robot2_initial_pos_j5)"
-    initial_pos_j6="$(arg robot2_initial_pos_j6)"/>
+    initial_pos_j6="$(arg robot2_initial_pos_j6)"
+    controller_config_file="${controller_config_file}"/>
   <xacro:welding_torch_macro prefix="robot2_"/>
   <joint name="robot2_tool0_to_torch" type="fixed">

File: hold_and_weld_description/urdf/robot1_gripper.xacro (robot description, xacro)
@@ -1,4 +1,4 @@
 <?xml version="1.0"?>
-<robot xmlns:xacro="http://ros.org/wiki/xacro" name="gp25_gripper_system">
+<robot xmlns:xacro="http://ros.org/wiki/xacro" name="gripper_system">
   <xacro:arg name="controller_config_file" default=""/>
   <xacro:property name="controller_config_file" value="$(arg controller_config_file)"/>
@@ -10,5 +10,5 @@
   <!-- Robot 1: Gripper System with Rail -->
   <xacro:linear_rail_macro parent="world" prefix="robot1_"/>
-  <xacro:gp25_arm_macro parent="robot1_rail_carriage" prefix="robot1_"/>
+  <xacro:gp25_arm_macro parent="robot1_rail_carriage" prefix="robot1_" controller_config_file="${controller_config_file}"/>
   <xacro:gripper_macro prefix="robot1_"/>
   <joint name="robot1_tool0_to_gripper" type="fixed">

File: hold_and_weld_description/urdf/robot2_welder.xacro (robot description, xacro)
@@ -1,12 +1,13 @@
 <?xml version="1.0"?>
-<robot xmlns:xacro="http://ros.org/wiki/xacro" name="gp25_welder_system">
+<robot xmlns:xacro="http://ros.org/wiki/xacro" name="welder_system">
   <xacro:arg name="controller_config_file" default=""/>
   <xacro:property name="controller_config_file" value="$(arg controller_config_file)"/>
   <!-- Include all macro files -->
-  <xacro:include filename="$(find hold_and_weld_description)/urdf/robots/gp25_arm_prefix.xacro"/>
+  <xacro:include filename="$(find hold_and_weld_description)/urdf/robots/ar2010_arm_prefix.xacro"/>
   <xacro:include filename="$(find hold_and_weld_description)/urdf/end_effectors/welding_torch_prefix.xacro"/>
   <link name="world"/>
   <!-- Robot 2: Welder System (standalone) -->
-  <xacro:gp25_arm_macro parent="world" prefix="robot2_" x="2.2" y="-0.5" z="0" yaw='3.14159'/>
+  <xacro:ar2010_arm_macro parent="world" prefix="robot2_" x="2.2" y="-0.5" z="0" yaw='3.14159'
+    controller_config_file="${controller_config_file}"/>
   <xacro:welding_torch_macro prefix="robot2_"/>
   <joint name="robot2_tool0_to_torch" type="fixed">

File: hold_and_weld_description/urdf/robots/ar2010_arm_prefix.xacro (robot description, xacro)
@@ -1,5 +1,5 @@
 <?xml version="1.0"?>
-<robot xmlns:xacro="http://ros.org/wiki/xacro" name="gp25_arm_macro">
-  <xacro:macro name="gp25_arm_macro"
+<robot xmlns:xacro="http://ros.org/wiki/xacro" name="ar2010_arm_macro">
+  <xacro:macro name="ar2010_arm_macro"
                params="parent prefix x:=0 y:=0 z:=0 roll:=0 pitch:=0 yaw:=0
                        initial_pos_j1:=0 initial_pos_j2:=0 initial_pos_j3:=0
@@ -12,12 +12,12 @@
       <origin xyz="${x} ${y} ${z}" rpy="${roll} ${pitch} ${yaw}"/>
     </joint>
-    <!-- Include the upstream Motoman GP25 kinematic description -->
-    <xacro:include filename="$(find hold_and_weld_description)/urdf/robots/gp25_macro.xacro"/>
-    <xacro:motoman_gp25 prefix="${prefix}"/>
+    <!-- Include the upstream Motoman AR2010 kinematic description -->
+    <xacro:include filename="$(find hold_and_weld_description)/urdf/robots/ar2010_macro.xacro"/>
+    <xacro:motoman_ar2010 prefix="${prefix}"/>
     <!-- Include the shared ros2_control block -->
     <xacro:include filename="$(find hold_and_weld_description)/urdf/robots/robot_arm_ros2_control.xacro"/>
     <xacro:robot_arm_ros2_control
       prefix="${prefix}"
-      ros2_control_name="${prefix}gp25_system"
+      ros2_control_name="${prefix}ar2010_system"
       initial_pos_j1="${initial_pos_j1}"
       initial_pos_j2="${initial_pos_j2}"
@@ -30,20 +30,20 @@
       <material>Gazebo/Blue</material>
     </gazebo>
-    <gazebo reference="${prefix}link_1_s">
+    <gazebo reference="${prefix}link_1">
       <material>Gazebo/Blue</material>
     </gazebo>
-    <gazebo reference="${prefix}link_2_l">
+    <gazebo reference="${prefix}link_2">
       <material>Gazebo/Blue</material>
     </gazebo>
-    <gazebo reference="${prefix}link_3_u">
+    <gazebo reference="${prefix}link_3">
       <material>Gazebo/Blue</material>
     </gazebo>
-    <gazebo reference="${prefix}link_4_r">
+    <gazebo reference="${prefix}link_4">
       <material>Gazebo/Blue</material>
     </gazebo>
-    <gazebo reference="${prefix}link_5_b">
+    <gazebo reference="${prefix}link_5">
       <material>Gazebo/Blue</material>
     </gazebo>
-    <gazebo reference="${prefix}link_6_t">
+    <gazebo reference="${prefix}link_6">
       <material>Gazebo/Blue</material>
     </gazebo>
