Commit message: add workcell configurator feature

File: hold_and_weld_description/urdf/dual_robot.xacro (robot description, xacro)
@@ -11,22 +11,24 @@
   <xacro:arg name="robot2_initial_pos_j5" default="0"/>
   <xacro:arg name="robot2_initial_pos_j6" default="0"/>
+  <!-- Slot models and poses; see config/workcell.yaml -->
+  <xacro:arg name="workcell_config" default="$(find hold_and_weld_description)/config/workcell.yaml"/>
+  <xacro:property name="workcell" value="${xacro.load_yaml('$(arg workcell_config)')}"/>
   <!-- Include all macro files -->
   <xacro:include filename="$(find hold_and_weld_description)/urdf/extra_axis/linear_rail_prefix.xacro"/>
-  <xacro:include filename="$(find hold_and_weld_description)/urdf/robots/gp25_arm_prefix.xacro"/> <!-- Robot1 (gripper) -->
-  <xacro:include filename="$(find hold_and_weld_description)/urdf/robots/gp25_arm_prefix.xacro"/> <!-- Robot2 (welder) -->
+  <xacro:include filename="$(find hold_and_weld_description)/urdf/robots/robot_catalog.xacro"/>
   <xacro:include filename="$(find hold_and_weld_description)/urdf/end_effectors/gripper_prefix.xacro"/>
   <xacro:include filename="$(find hold_and_weld_description)/urdf/end_effectors/welding_torch_prefix.xacro"/>
   <link name="world"/>
   <!-- Robot 1: Gripper System with Rail -->
-  <xacro:linear_rail_macro parent="world" prefix="robot1_"/>
-  <xacro:gp25_arm_macro parent="robot1_rail_carriage" prefix="robot1_" controller_config_file="${controller_config_file}"/>
-  <xacro:gripper_macro prefix="robot1_"/>
-  <joint name="robot1_tool0_to_gripper" type="fixed">
-    <parent link="robot1_tool0"/>
-    <child link="robot1_gripper_base"/>
-    <origin xyz="0 0 0.025" rpy="3.14159 0 0"/>
-  </joint>
+  <xacro:property name="robot1" value="${workcell['robots']['robot1']}"/>
+  <xacro:linear_rail_macro parent="world" prefix="robot1_"
+    x="${robot1['x']}" y="${robot1['y']}" z="${robot1['z']}" yaw="${robot1['yaw']}"/>
+  <xacro:robot_arm_macro model="${robot1['model']}" parent="robot1_rail_carriage" prefix="robot1_"
+    controller_config_file="${controller_config_file}"/>
+  <xacro:gripper_macro prefix="robot1_" parent="robot1_tool0"/>
   <!-- Robot 2: Welder System (standalone) -->
-  <xacro:gp25_arm_macro parent="world" prefix="robot2_" x="2.2" y="-0.5" z="0" yaw='3.14159'
+  <xacro:property name="robot2" value="${workcell['robots']['robot2']}"/>
+  <xacro:robot_arm_macro model="${robot2['model']}" parent="world" prefix="robot2_"
+    x="${robot2['x']}" y="${robot2['y']}" z="${robot2['z']}" yaw="${robot2['yaw']}"
     initial_pos_j1="$(arg robot2_initial_pos_j1)"
     initial_pos_j2="$(arg robot2_initial_pos_j2)"

File: hold_and_weld_description/urdf/end_effectors/gripper_prefix.xacro (robot description, xacro)
@@ -10,6 +10,8 @@
     - finger elements: Each movable finger with its controlling joint
     - Joints must be prismatic type with axis and limits defined
+    - The mount joint to `parent` carries this gripper's coupling offset, so a
+      gripper swap stays inside this file
   -->
-  <xacro:macro name="gripper_macro" params="prefix">
+  <xacro:macro name="gripper_macro" params="prefix parent">
     <!-- This section is parsed by GripperParser to extract gripper kinematics -->
     <gripper_metadata>
@@ -27,4 +29,9 @@
       <tcp_offset xyz="0 0 -0.12" rpy="0 0 0"/>
     </gripper_metadata>
+    <joint name="${prefix}tool0_to_gripper" type="fixed">
+      <parent link="${parent}"/>
+      <child link="${prefix}gripper_base"/>
+      <origin xyz="0 0 0.025" rpy="3.14159 0 0"/>
+    </joint>
     <link name="${prefix}gripper_base">
       <visual>

File: hold_and_weld_description/urdf/extra_axis/linear_rail_prefix.xacro (robot description, xacro)
@@ -1,5 +1,5 @@
 <?xml version="1.0"?>
 <robot xmlns:xacro="http://ros.org/wiki/xacro" name="linear_rail">
-  <xacro:macro name="linear_rail_macro" params="parent prefix">
+  <xacro:macro name="linear_rail_macro" params="parent prefix x:=0 y:=0 z:=0 yaw:=0">
     <xacro:property name="rail_height" value="0.2"/>
     <xacro:property name="rail_length" value="4.0"/>
@@ -30,5 +30,5 @@
       <parent link="${parent}"/>
       <child link="${prefix}rail_base"/>
-      <origin xyz="0 0 0" rpy="0 0 0"/>
+      <origin xyz="${x} ${y} ${z}" rpy="0 0 ${yaw}"/>
     </joint>
     <link name="${prefix}rail_carriage">

File: hold_and_weld_description/urdf/robot1_gripper.xacro (robot description, xacro)
@@ -3,18 +3,19 @@
   <xacro:arg name="controller_config_file" default=""/>
   <xacro:property name="controller_config_file" value="$(arg controller_config_file)"/>
+  <!-- Slot models and poses; see config/workcell.yaml -->
+  <xacro:arg name="workcell_config" default="$(find hold_and_weld_description)/config/workcell.yaml"/>
+  <xacro:property name="workcell" value="${xacro.load_yaml('$(arg workcell_config)')}"/>
   <!-- Include all macro files -->
   <xacro:include filename="$(find hold_and_weld_description)/urdf/extra_axis/linear_rail_prefix.xacro"/>
-  <xacro:include filename="$(find hold_and_weld_description)/urdf/robots/gp25_arm_prefix.xacro"/>
+  <xacro:include filename="$(find hold_and_weld_description)/urdf/robots/robot_catalog.xacro"/>
   <xacro:include filename="$(find hold_and_weld_description)/urdf/end_effectors/gripper_prefix.xacro"/>
   <link name="world"/>
   <!-- Robot 1: Gripper System with Rail -->
-  <xacro:linear_rail_macro parent="world" prefix="robot1_"/>
-  <xacro:gp25_arm_macro parent="robot1_rail_carriage" prefix="robot1_" controller_config_file="${controller_config_file}"/>
-  <xacro:gripper_macro prefix="robot1_"/>
-  <joint name="robot1_tool0_to_gripper" type="fixed">
-    <parent link="robot1_tool0"/>
-    <child link="robot1_gripper_base"/>
-    <origin xyz="0 0 0.025" rpy="3.14159 0 0"/>
-  </joint>
+  <xacro:property name="robot1" value="${workcell['robots']['robot1']}"/>
+  <xacro:linear_rail_macro parent="world" prefix="robot1_"
+    x="${robot1['x']}" y="${robot1['y']}" z="${robot1['z']}" yaw="${robot1['yaw']}"/>
+  <xacro:robot_arm_macro model="${robot1['model']}" parent="robot1_rail_carriage" prefix="robot1_"
+    controller_config_file="${controller_config_file}"/>
+  <xacro:gripper_macro prefix="robot1_" parent="robot1_tool0"/>
   <gazebo>
     <plugin filename="gz_ros2_control-system" name="gz_ros2_control::GazeboSimROS2ControlPlugin">

File: hold_and_weld_description/urdf/robot2_welder.xacro (robot description, xacro)
@@ -3,11 +3,15 @@
   <xacro:arg name="controller_config_file" default=""/>
   <xacro:property name="controller_config_file" value="$(arg controller_config_file)"/>
+  <!-- Slot models and poses; see config/workcell.yaml -->
+  <xacro:arg name="workcell_config" default="$(find hold_and_weld_description)/config/workcell.yaml"/>
+  <xacro:property name="workcell" value="${xacro.load_yaml('$(arg workcell_config)')}"/>
   <!-- Include all macro files -->
-  <xacro:include filename="$(find hold_and_weld_description)/urdf/robots/gp25_arm_prefix.xacro"/>
+  <xacro:include filename="$(find hold_and_weld_description)/urdf/robots/robot_catalog.xacro"/>
   <xacro:include filename="$(find hold_and_weld_description)/urdf/end_effectors/welding_torch_prefix.xacro"/>
   <link name="world"/>
-  <!-- Robot 2: Welder System (standalone). Matches dual_robot.xacro, which uses
-       gp25 for both robots (see commit "Taking back to gp25"). -->
-  <xacro:gp25_arm_macro parent="world" prefix="robot2_" x="2.2" y="-0.5" z="0" yaw='3.14159'
+  <!-- Robot 2: Welder System (standalone). Same slot as in dual_robot.xacro. -->
+  <xacro:property name="robot2" value="${workcell['robots']['robot2']}"/>
+  <xacro:robot_arm_macro model="${robot2['model']}" parent="world" prefix="robot2_"
+    x="${robot2['x']}" y="${robot2['y']}" z="${robot2['z']}" yaw="${robot2['yaw']}"
     controller_config_file="${controller_config_file}"/>
   <xacro:welding_torch_macro prefix="robot2_"/>

Commit message: add gripper adding gripper catalogue, add new grippers, workcell configurator io change

File: hold_and_weld_description/urdf/dual_robot.xacro (robot description, xacro)
@@ -17,5 +17,5 @@
   <xacro:include filename="$(find hold_and_weld_description)/urdf/extra_axis/linear_rail_prefix.xacro"/>
   <xacro:include filename="$(find hold_and_weld_description)/urdf/robots/robot_catalog.xacro"/>
-  <xacro:include filename="$(find hold_and_weld_description)/urdf/end_effectors/gripper_prefix.xacro"/>
+  <xacro:include filename="$(find hold_and_weld_description)/urdf/end_effectors/gripper_catalog.xacro"/>
   <xacro:include filename="$(find hold_and_weld_description)/urdf/end_effectors/welding_torch_prefix.xacro"/>
   <link name="world"/>
@@ -26,5 +26,5 @@
   <xacro:robot_arm_macro model="${robot1['model']}" parent="robot1_rail_carriage" prefix="robot1_"
     controller_config_file="${controller_config_file}"/>
-  <xacro:gripper_macro prefix="robot1_" parent="robot1_tool0"/>
+  <xacro:gripper_catalog_macro model="${workcell.get('gripper_model', '')}" prefix="robot1_" parent="robot1_tool0"/>
   <!-- Robot 2: Welder System (standalone) -->
   <xacro:property name="robot2" value="${workcell['robots']['robot2']}"/>

File: hold_and_weld_description/urdf/end_effectors/gripper_prefix.xacro (robot description, xacro)
@@ -2,15 +2,10 @@
 <robot xmlns:xacro="http://ros.org/wiki/xacro" name="gp25_gripper">
   <!--
-    Gripper Convention Template
-    This URDF follows the hold_and_weld gripper convention.
-    The gripper_metadata section below is parsed by GripperParser
-    to extract kinematic information for grasp planning.
-    Required elements:
-    - base_link: The static palm/base of the gripper
-    - finger elements: Each movable finger with its controlling joint
-    - Joints must be prismatic type with axis and limits defined
-    - The mount joint to `parent` carries this gripper's coupling offset, so a
-      gripper swap stays inside this file
+    Placeholder gripper: the "placeholder" entry of gripper_catalog.xacro, which
+    documents the canonical interface every gripper model follows. The
+    gripper_metadata section below is parsed by GripperParser for grasp planning.
   -->
+  <xacro:property name="placeholder_travel" value="0.15"/>
+  <xacro:property name="placeholder_spawn_position" value="${placeholder_travel / 2}"/>
   <xacro:macro name="gripper_macro" params="prefix parent">
     <!-- This section is parsed by GripperParser to extract gripper kinematics -->
@@ -103,6 +98,6 @@
       <origin xyz="0 0.03 -0.02" rpy="0 0 0"/>
       <axis xyz="0 1 0"/>
-      <limit lower="0.0" upper="0.15" effort="100" velocity="0.1"/>
-      <dynamics damping="1.0" friction="2.0"/>
+      <limit lower="0.0" upper="${placeholder_travel}" effort="100" velocity="0.1"/>
+      <dynamics damping="1.0" friction="0.0"/>
     </joint>
     <joint name="${prefix}right_finger_joint" type="prismatic">
@@ -111,6 +106,6 @@
       <origin xyz="0 -0.03 -0.02" rpy="0 0 0"/>
       <axis xyz="0 -1 0"/>
-      <limit lower="0.0" upper="0.15" effort="100" velocity="0.1"/>
-      <dynamics damping="1.0" friction="2.0"/>
+      <limit lower="0.0" upper="${placeholder_travel}" effort="100" velocity="0.1"/>
+      <dynamics damping="1.0" friction="0.0"/>
     </joint>
     <gazebo reference="${prefix}gripper_base">
@@ -136,7 +131,9 @@
         <command_interface name="position">
           <param name="min">0.0</param>
-          <param name="max">0.15</param>
+          <param name="max">${placeholder_travel}</param>
         </command_interface>
-        <state_interface name="position"/>
+        <state_interface name="position">
+          <param name="initial_value">${placeholder_spawn_position}</param>
+        </state_interface>
         <state_interface name="velocity"/>
       </joint>
@@ -144,7 +141,9 @@
         <command_interface name="position">
           <param name="min">0.0</param>
-          <param name="max">0.15</param>
+          <param name="max">${placeholder_travel}</param>
         </command_interface>
-        <state_interface name="position"/>
+        <state_interface name="position">
+          <param name="initial_value">${placeholder_spawn_position}</param>
+        </state_interface>
         <state_interface name="velocity"/>
       </joint>

File: hold_and_weld_description/urdf/robot1_gripper.xacro (robot description, xacro)
@@ -9,5 +9,5 @@
   <xacro:include filename="$(find hold_and_weld_description)/urdf/extra_axis/linear_rail_prefix.xacro"/>
   <xacro:include filename="$(find hold_and_weld_description)/urdf/robots/robot_catalog.xacro"/>
-  <xacro:include filename="$(find hold_and_weld_description)/urdf/end_effectors/gripper_prefix.xacro"/>
+  <xacro:include filename="$(find hold_and_weld_description)/urdf/end_effectors/gripper_catalog.xacro"/>
   <link name="world"/>
   <!-- Robot 1: Gripper System with Rail -->
@@ -17,5 +17,5 @@
   <xacro:robot_arm_macro model="${robot1['model']}" parent="robot1_rail_carriage" prefix="robot1_"
     controller_config_file="${controller_config_file}"/>
-  <xacro:gripper_macro prefix="robot1_" parent="robot1_tool0"/>
+  <xacro:gripper_catalog_macro model="${workcell.get('gripper_model', '')}" prefix="robot1_" parent="robot1_tool0"/>
   <gazebo>
     <plugin filename="gz_ros2_control-system" name="gz_ros2_control::GazeboSimROS2ControlPlugin">

Commit message: Change default scenario and comment back old version

File: hold_and_weld_description/urdf/dual_robot.xacro (robot description, xacro)
@@ -3,4 +3,12 @@
   <xacro:arg name="controller_config_file" default=""/>
   <xacro:property name="controller_config_file" value="$(arg controller_config_file)"/>
+  <!-- Robot1 initial joint positions (radians). Populated by sim_gazebo.launch.py
+       from pick_place_targets.yaml start_pose so the gripper arm spawns collision-free. -->
+  <xacro:arg name="robot1_initial_pos_j1" default="0"/>
+  <xacro:arg name="robot1_initial_pos_j2" default="0"/>
+  <xacro:arg name="robot1_initial_pos_j3" default="0"/>
+  <xacro:arg name="robot1_initial_pos_j4" default="0"/>
+  <xacro:arg name="robot1_initial_pos_j5" default="0"/>
+  <xacro:arg name="robot1_initial_pos_j6" default="0"/>
   <!-- Robot2 initial joint positions (radians). Populated by sim_gazebo.launch.py
        from welding.yaml safety_pose so the welder spawns collision-free. -->
@@ -11,4 +19,7 @@
   <xacro:arg name="robot2_initial_pos_j5" default="0"/>
   <xacro:arg name="robot2_initial_pos_j6" default="0"/>
+  <!-- Gazebo model name of the part robot1 grasps (objects.yaml child_link spawn_name).
+       Populated by sim_gazebo.launch.py; empty leaves the Gazebo grasp joint out. -->
+  <xacro:arg name="grasp_object_model" default=""/>
   <!-- Slot models and poses; see config/workcell.yaml -->
   <xacro:arg name="workcell_config" default="$(find hold_and_weld_description)/config/workcell.yaml"/>
@@ -25,6 +36,13 @@
     x="${robot1['x']}" y="${robot1['y']}" z="${robot1['z']}" yaw="${robot1['yaw']}"/>
   <xacro:robot_arm_macro model="${robot1['model']}" parent="robot1_rail_carriage" prefix="robot1_"
+    initial_pos_j1="$(arg robot1_initial_pos_j1)"
+    initial_pos_j2="$(arg robot1_initial_pos_j2)"
+    initial_pos_j3="$(arg robot1_initial_pos_j3)"
+    initial_pos_j4="$(arg robot1_initial_pos_j4)"
+    initial_pos_j5="$(arg robot1_initial_pos_j5)"
+    initial_pos_j6="$(arg robot1_initial_pos_j6)"
     controller_config_file="${controller_config_file}"/>
-  <xacro:gripper_catalog_macro model="${workcell.get('gripper_model', '')}" prefix="robot1_" parent="robot1_tool0"/>
+  <xacro:gripper_catalog_macro model="${workcell.get('gripper_model', '')}" prefix="robot1_" parent="robot1_tool0"
+    grasp_object_model="$(arg grasp_object_model)"/>
   <!-- Robot 2: Welder System (standalone) -->
   <xacro:property name="robot2" value="${workcell['robots']['robot2']}"/>

File: hold_and_weld_description/urdf/end_effectors/gripper_catalog.xacro (robot description, xacro)
@@ -38,5 +38,5 @@
   <xacro:include filename="$(find hold_and_weld_description)/urdf/end_effectors/robotiq_2f_140_gripper_prefix.xacro"/>
   <xacro:property name="gripper_catalog" value="${['placeholder', 'rethink_electric', 'schunk_pg70', 'onrobot_2fg7', 'robotiq_2f_140']}"/>
-  <xacro:macro name="gripper_catalog_macro" params="model prefix parent">
+  <xacro:macro name="gripper_catalog_macro" params="model prefix parent grasp_object_model:=''">
     <xacro:if value="${model == ''}">
       ${xacro.fatal('workcell.yaml has no gripper_model for', prefix, '- set it to one of', gripper_catalog)}
@@ -60,4 +60,21 @@
       <xacro:robotiq_2f_140_gripper_macro prefix="${prefix}" parent="${parent}"/>
     </xacro:if>
+    <!--
+      Attaches as soon as the part spawns; the gripper action server detaches it first.
+      Parent is link_6: URDF to SDF lumps the fixed gripper chain into it.
+    -->
+    <xacro:if value="${grasp_object_model != ''}">
+      <gazebo>
+        <plugin filename="gz-sim-detachable-joint-system" name="gz::sim::systems::DetachableJoint">
+          <parent_link>${prefix}link_6</parent_link>
+          <child_model>${grasp_object_model}</child_model>
+          <child_link>child_link</child_link>
+          <attach_topic>/${prefix}grasp/attach</attach_topic>
+          <detach_topic>/${prefix}grasp/detach</detach_topic>
+          <output_topic>/${prefix}grasp/state</output_topic>
+          <suppress_child_warning>true</suppress_child_warning>
+        </plugin>
+      </gazebo>
+    </xacro:if>
   </xacro:macro>
 </robot>

File: hold_and_weld_description/urdf/environment/robotiq_cube.urdf.xacro (robot description, xacro)
@@ -50,6 +50,7 @@
       </surface>
     </collision>
-  <gravity>0</gravity>
-  <static>true</static>
+    <!-- Gravity on, not static: the cube rests on
+         the floor (pick) or the table top (end_pose) so a finger touching first
+         cannot float it away, and the grasp DetachableJoint carries it once attached. -->
   </gazebo>
 </robot>

File: hold_and_weld_description/urdf/robot1_gripper.xacro (robot description, xacro)
@@ -3,4 +3,15 @@
   <xacro:arg name="controller_config_file" default=""/>
   <xacro:property name="controller_config_file" value="$(arg controller_config_file)"/>
+  <!-- Robot1 initial joint positions (radians). Populated by sim_gazebo.launch.py
+       from pick_place_targets.yaml start_pose so the gripper arm spawns collision-free. -->
+  <xacro:arg name="robot1_initial_pos_j1" default="0"/>
+  <xacro:arg name="robot1_initial_pos_j2" default="0"/>
+  <xacro:arg name="robot1_initial_pos_j3" default="0"/>
+  <xacro:arg name="robot1_initial_pos_j4" default="0"/>
+  <xacro:arg name="robot1_initial_pos_j5" default="0"/>
+  <xacro:arg name="robot1_initial_pos_j6" default="0"/>
+  <!-- Gazebo model name of the part robot1 grasps (objects.yaml child_link spawn_name).
+       Populated by sim_gazebo.launch.py; empty leaves the Gazebo grasp joint out. -->
+  <xacro:arg name="grasp_object_model" default=""/>
   <!-- Slot models and poses; see config/workcell.yaml -->
   <xacro:arg name="workcell_config" default="$(find hold_and_weld_description)/config/workcell.yaml"/>
@@ -16,6 +27,13 @@
     x="${robot1['x']}" y="${robot1['y']}" z="${robot1['z']}" yaw="${robot1['yaw']}"/>
   <xacro:robot_arm_macro model="${robot1['model']}" parent="robot1_rail_carriage" prefix="robot1_"
+    initial_pos_j1="$(arg robot1_initial_pos_j1)"
+    initial_pos_j2="$(arg robot1_initial_pos_j2)"
+    initial_pos_j3="$(arg robot1_initial_pos_j3)"
+    initial_pos_j4="$(arg robot1_initial_pos_j4)"
+    initial_pos_j5="$(arg robot1_initial_pos_j5)"
+    initial_pos_j6="$(arg robot1_initial_pos_j6)"
     controller_config_file="${controller_config_file}"/>
-  <xacro:gripper_catalog_macro model="${workcell.get('gripper_model', '')}" prefix="robot1_" parent="robot1_tool0"/>
+  <xacro:gripper_catalog_macro model="${workcell.get('gripper_model', '')}" prefix="robot1_" parent="robot1_tool0"
+    grasp_object_model="$(arg grasp_object_model)"/>
   <gazebo>
     <plugin filename="gz_ros2_control-system" name="gz_ros2_control::GazeboSimROS2ControlPlugin">

File: hold_and_weld_description/urdf/robots/robot_catalog.xacro (robot description, xacro)
@@ -10,5 +10,7 @@
   <xacro:include filename="$(find hold_and_weld_description)/urdf/robots/gp25_arm_prefix.xacro"/>
   <xacro:include filename="$(find hold_and_weld_description)/urdf/robots/ar2010_arm_prefix.xacro"/>
-  <xacro:property name="robot_catalog" value="${['gp25', 'ar2010']}"/>
+  <xacro:include filename="$(find hold_and_weld_description)/urdf/robots/hc10dt_arm_prefix.xacro"/>
+  <xacro:include filename="$(find hold_and_weld_description)/urdf/robots/gp8l_arm_prefix.xacro"/>
+  <xacro:property name="robot_catalog" value="${['gp25', 'ar2010', 'hc10dt', 'gp8l']}"/>
   <xacro:macro name="robot_arm_macro"
                params="model parent prefix x:=0 y:=0 z:=0 yaw:=0
@@ -33,4 +35,18 @@
         controller_config_file="${controller_config_file}"/>
     </xacro:if>
+    <xacro:if value="${model == 'hc10dt'}">
+      <xacro:hc10dt_arm_macro parent="${parent}" prefix="${prefix}" x="${x}" y="${y}" z="${z}" yaw="${yaw}"
+        initial_pos_j1="${initial_pos_j1}" initial_pos_j2="${initial_pos_j2}"
+        initial_pos_j3="${initial_pos_j3}" initial_pos_j4="${initial_pos_j4}"
+        initial_pos_j5="${initial_pos_j5}" initial_pos_j6="${initial_pos_j6}"
+        controller_config_file="${controller_config_file}"/>
+    </xacro:if>
+    <xacro:if value="${model == 'gp8l'}">
+      <xacro:gp8l_arm_macro parent="${parent}" prefix="${prefix}" x="${x}" y="${y}" z="${z}" yaw="${yaw}"
+        initial_pos_j1="${initial_pos_j1}" initial_pos_j2="${initial_pos_j2}"
+        initial_pos_j3="${initial_pos_j3}" initial_pos_j4="${initial_pos_j4}"
+        initial_pos_j5="${initial_pos_j5}" initial_pos_j6="${initial_pos_j6}"
+        controller_config_file="${controller_config_file}"/>
+    </xacro:if>
   </xacro:macro>
 </robot>
